File: hardware/mainboard/analogins.sch (KiCad schematic (older format))
At the start: 19 parts, among them U13 MCP6004

Commit message: start to change to tht!
Parts:
- C37, C38, C39, C40: footprint Capacitor_SMD:C_0603_1608Metric_Pad1.05x0.95mm_HandSolder -> Sonosus:Capacitor_NonPolarized
- C42, C43: footprint Capacitor_SMD:C_0603_1608Metric_Pad1.05x0.95mm_HandSolder -> Sonosus:Capacitor_NonPolarizedSmall
- R48, R49, R50, R51, R52, R53, R54, R55, R56, R57, R58, R59: footprint Resistor_SMD:R_0603_1608Metric_Pad1.05x0.95mm_HandSolder -> Sonosus:Resistor
Changed lines of the file:
@@
 F 0 "R48" V 1295 1250 50  0000 C CNN
 F 1 "100k" V 1386 1250 50  0000 C CNN
-F 2 "Resistor_SMD:R_0603_1608Metric_Pad1.05x0.95mm_HandSolder" V 1540 1240 50  0001 C CNN
+F 2 "Sonosus:Resistor" V 1540 1240 50  0001 C CNN
 F 3 "~" H 1500 1250 50  0001 C CNN
 F 4 "yes" H 1500 1250 50  0001 C CNN "finalized"
@@
 F 0 "R49" V 1295 1550 50  0000 C CNN
 F 1 "169k" V 1386 1550 50  0000 C CNN
-F 2 "Resistor_SMD:R_0603_1608Metric_Pad1.05x0.95mm_HandSolder" V 1540 1540 50  0001 C CNN
+F 2 "Sonosus:Resistor" V 1540 1540 50  0001 C CNN
 F 3 "~" H 1500 1550 50  0001 C CNN
 F 4 "yes" H 1500 1550 50  0001 C CNN "finalized"
@@
 F 0 "R56" V 2195 1650 50  0000 C CNN
 F 1 "56k" V 2286 1650 50  0000 C CNN
-F 2 "Resistor_SMD:R_0603_1608Metric_Pad1.05x0.95mm_HandSolder" V 2440 1640 50  0001 C CNN
+F 2 "Sonosus:Resistor" V 2440 1640 50  0001 C CNN
 F 3 "~" H 2400 1650 50  0001 C CNN
 F 4 "yes" H 2400 1650 50  0001 C CNN "finalized"
@@
 F 0 "C37" V 2629 2000 50  0000 C CNN
 F 1 "2.2nF" V 2538 2000 50  0000 C CNN
-F 2 "Capacitor_SMD:C_0603_1608Metric_Pad1.05x0.95mm_HandSolder" H 2400 2000 50  0001 C CNN
+F 2 "Sonosus:Capacitor_NonPolarized" H 2400 2000 50  0001 C CNN
 F 3 "~" H 2400 2000 50  0001 C CNN
 F 4 "yes" H 2400 2000 50  0001 C CNN "finalized"
@@
 F 0 "R50" V 1295 2750 50  0000 C CNN
 F 1 "100k" V 1386 2750 50  0000 C CNN
-F 2 "Resistor_SMD:R_0603_1608Metric_Pad1.05x0.95mm_HandSolder" V 1540 2740 50  0001 C CNN
+F 2 "Sonosus:Resistor" V 1540 2740 50  0001 C CNN
 F 3 "~" H 1500 2750 50  0001 C CNN
 F 4 "yes" H 1500 2750 50  0001 C CNN "finalized"
@@
 F 0 "R51" V 1295 3050 50  0000 C CNN
 F 1 "169k" V 1386 3050 50  0000 C CNN
-F 2 "Resistor_SMD:R_0603_1608Metric_Pad1.05x0.95mm_HandSolder" V 1540 3040 50  0001 C CNN
+F 2 "Sonosus:Resistor" V 1540 3040 50  0001 C CNN
 F 3 "~" H 1500 3050 50  0001 C CNN
 F 4 "yes" H 1500 3050 50  0001 C CNN "finalized"
@@
 F 0 "R57" V 2195 3150 50  0000 C CNN
 F 1 "56k" V 2286 3150 50  0000 C CNN
-F 2 "Resistor_SMD:R_0603_1608Metric_Pad1.05x0.95mm_HandSolder" V 2440 3140 50  0001 C CNN
+F 2 "Sonosus:Resistor" V 2440 3140 50  0001 C CNN
 F 3 "~" H 2400 3150 50  0001 C CNN
 F 4 "yes" H 2400 3150 50  0001 C CNN "finalized"
@@
 F 0 "C38" V 2629 3500 50  0000 C CNN
 F 1 "2.2nF" V 2538 3500 50  0000 C CNN
-F 2 "Capacitor_SMD:C_0603_1608Metric_Pad1.05x0.95mm_HandSolder" H 2400 3500 50  0001 C CNN
+F 2 "Sonosus:Capacitor_NonPolarized" H 2400 3500 50  0001 C CNN
 F 3 "~" H 2400 3500 50  0001 C CNN
 F 4 "yes" H 2400 3500 50  0001 C CNN "finalized"
@@
 F 0 "R52" V 1295 4200 50  0000 C CNN
 F 1 "100k" V 1386 4200 50  0000 C CNN
-F 2 "Resistor_SMD:R_0603_1608Metric_Pad1.05x0.95mm_HandSolder" V 1540 4190 50  0001 C CNN
+F 2 "Sonosus:Resistor" V 1540 4190 50  0001 C CNN
 F 3 "~" H 1500 4200 50  0001 C CNN
 F 4 "yes" H 1500 4200 50  0001 C CNN "finalized"
@@
 F 0 "R53" V 1295 4500 50  0000 C CNN
 F 1 "200k" V 1386 4500 50  0000 C CNN
-F 2 "Resistor_SMD:R_0603_1608Metric_Pad1.05x0.95mm_HandSolder" V 1540 4490 50  0001 C CNN
+F 2 "Sonosus:Resistor" V 1540 4490 50  0001 C CNN
 F 3 "~" H 1500 4500 50  0001 C CNN
 F 4 "yes" H 1500 4500 50  0001 C CNN "finalized"
@@
 F 0 "R58" V 2195 4600 50  0000 C CNN
 F 1 "64.9k" V 2286 4600 50  0000 C CNN
-F 2 "Resistor_SMD:R_0603_1608Metric_Pad1.05x0.95mm_HandSolder" V 2440 4590 50  0001 C CNN
+F 2 "Sonosus:Resistor" V 2440 4590 50  0001 C CNN
 F 3 "~" H 2400 4600 50  0001 C CNN
 F 4 "yes" H 2400 4600 50  0001 C CNN "finalized"
@@
 F 0 "C39" V 2629 4950 50  0000 C CNN
 F 1 "4.7nF" V 2538 4950 50  0000 C CNN
-F 2 "Capacitor_SMD:C_0603_1608Metric_Pad1.05x0.95mm_HandSolder" H 2400 4950 50  0001 C CNN
+F 2 "Sonosus:Capacitor_NonPolarized" H 2400 4950 50  0001 C CNN
 F 3 "~" H 2400 4950 50  0001 C CNN
 F 4 "yes" H 2400 4950 50  0001 C CNN "finalized"
@@
 F 0 "R54" V 1295 5650 50  0000 C CNN
 F 1 "100k" V 1386 5650 50  0000 C CNN
-F 2 "Resistor_SMD:R_0603_1608Metric_Pad1.05x0.95mm_HandSolder" V 1540 5640 50  0001 C CNN
+F 2 "Sonosus:Resistor" V 1540 5640 50  0001 C CNN
 F 3 "~" H 1500 5650 50  0001 C CNN
 F 4 "yes" H 1500 5650 50  0001 C CNN "finalized"
@@
 F 0 "R55" V 1295 5950 50  0000 C CNN
 F 1 "200k" V 1386 5950 50  0000 C CNN
-F 2 "Resistor_SMD:R_0603_1608Metric_Pad1.05x0.95mm_HandSolder" V 1540 5940 50  0001 C CNN
+F 2 "Sonosus:Resistor" V 1540 5940 50  0001 C CNN
 F 3 "~" H 1500 5950 50  0001 C CNN
 F 4 "yes" H 1500 5950 50  0001 C CNN "finalized"
@@
 F 0 "R59" V 2195 6050 50  0000 C CNN
 F 1 "64.9k" V 2286 6050 50  0000 C CNN
-F 2 "Resistor_SMD:R_0603_1608Metric_Pad1.05x0.95mm_HandSolder" V 2440 6040 50  0001 C CNN
+F 2 "Sonosus:Resistor" V 2440 6040 50  0001 C CNN
 F 3 "~" H 2400 6050 50  0001 C CNN
 F 4 "yes" H 2400 6050 50  0001 C CNN "finalized"
@@
 F 0 "C40" V 2629 6400 50  0000 C CNN
 F 1 "4.7nF" V 2538 6400 50  0000 C CNN
-F 2 "Capacitor_SMD:C_0603_1608Metric_Pad1.05x0.95mm_HandSolder" H 2400 6400 50  0001 C CNN
+F 2 "Sonosus:Capacitor_NonPolarized" H 2400 6400 50  0001 C CNN
 F 3 "~" H 2400 6400 50  0001 C CNN
 F 4 "yes" H 2400 6400 50  0001 C CNN "finalized"
@@
 F 0 "C42" H 8258 5954 50  0000 R CNN
 F 1 "0.1uF" H 8258 6045 50  0000 R CNN
-F 2 "Capacitor_SMD:C_0603_1608Metric_Pad1.05x0.95mm_HandSolder" H 8350 6000 50  0001 C CNN
+F 2 "Sonosus:Capacitor_NonPolarizedSmall" H 8350 6000 50  0001 C CNN
 F 3 "~" H 8350 6000 50  0001 C CNN
 F 4 "yes" H 8350 6000 50  0001 C CNN "finalized"
@@
 F 0 "C43" H 8858 5954 50  0000 R CNN
 F 1 "0.1uF" H 8858 6045 50  0000 R CNN
-F 2 "Capacitor_SMD:C_0603_1608Metric_Pad1.05x0.95mm_HandSolder" H 8950 6000 50  0001 C CNN
+F 2 "Sonosus:Capacitor_NonPolarizedSmall" H 8950 6000 50  0001 C CNN
 F 3 "~" H 8950 6000 50  0001 C CNN
 F 4 "yes" H 8950 6000 50  0001 C CNN "finalized"
