File: hardware/mainboard/castor.sch (KiCad schematic (older format))
At the start: 42 parts, among them Q1 MMBT3906, U3 TL074, U4 74LVC2G74, U5 MCP6001-OT, U6 TL074

Commit message: start to change to tht!
Parts:
- C10, C5, C7, C8: footprint Capacitor_SMD:C_0603_1608Metric_Pad1.05x0.95mm_HandSolder -> Sonosus:Capacitor_NonPolarizedSmall
- C11, C12, C13: footprint Capacitor_SMD:C_0805_2012Metric_Pad1.15x1.40mm_HandSolder -> Capacitor_THT:C_Disc_D4.3mm_W1.9mm_P5.00mm
- C14, C15, C16, C17, C6, C9: footprint Capacitor_SMD:C_0603_1608Metric_Pad1.05x0.95mm_HandSolder -> Sonosus:Capacitor_NonPolarized
- R10, R11, R12, R13, R14, R15, R16, R17, R18, R19, R2, R20, R21, R22, R23, R3, R4, R5, R6, R61, R7, R8, R9: footprint Resistor_SMD:R_0603_1608Metric_Pad1.05x0.95mm_HandSolder -> Sonosus:Resistor
