File: hardware/mainboard/mcu.sch (KiCad schematic (older format))
At the start: 20 parts, among them J2 Tag-Connect SWD, J3 USB_MICRO_RIGHT, SW1 RESET, U7 ATSAMD21G18A-AUT, U8 MCP4728

Commit message: start to change to tht!
Parts:
- C18: footprint Capacitor_SMD:C_0603_1608Metric_Pad1.05x0.95mm_HandSolder -> Sonosus:Capacitor_NonPolarized
- C19, C20, C21, C22, C49, C50: footprint Capacitor_SMD:C_0603_1608Metric_Pad1.05x0.95mm_HandSolder -> Sonosus:Capacitor_NonPolarizedSmall
- C23: footprint Capacitor_SMD:C_0805_2012Metric_Pad1.15x1.40mm_HandSolder -> Capacitor_THT:C_Disc_D4.3mm_W1.9mm_P5.00mm
- R24, R25: footprint Resistor_SMD:R_0603_1608Metric_Pad1.05x0.95mm_HandSolder -> Sonosus:Resistor
Changed lines of the file:
@@
 F 0 "C18" H 3165 1696 50  0000 L CNN
 F 1 "1uF" H 3165 1605 50  0000 L CNN
-F 2 "Capacitor_SMD:C_0603_1608Metric_Pad1.05x0.95mm_HandSolder" H 3088 1500 50  0001 C CNN
+F 2 "Sonosus:Capacitor_NonPolarized" H 3088 1500 50  0001 C CNN
 F 3 "~" H 3050 1650 50  0001 C CNN
 F 4 "yes" H 3050 1650 50  0001 C CNN "finalized"
@@
 F 0 "C19" H 3265 7046 50  0000 L CNN
 F 1 "0.1uF" H 3265 6955 50  0000 L CNN
-F 2 "Capacitor_SMD:C_0603_1608Metric_Pad1.05x0.95mm_HandSolder" H 3188 6850 50  0001 C CNN
+F 2 "Sonosus:Capacitor_NonPolarizedSmall" H 3188 6850 50  0001 C CNN
 F 3 "~" H 3150 7000 50  0001 C CNN
 F 4 "yes" H 3150 7000 50  0001 C CNN "finalized"
@@
 F 0 "C20" H 3765 7046 50  0000 L CNN
 F 1 "0.1uF" H 3765 6955 50  0000 L CNN
-F 2 "Capacitor_SMD:C_0603_1608Metric_Pad1.05x0.95mm_HandSolder" H 3688 6850 50  0001 C CNN
+F 2 "Sonosus:Capacitor_NonPolarizedSmall" H 3688 6850 50  0001 C CNN
 F 3 "~" H 3650 7000 50  0001 C CNN
 F 4 "yes" H 3650 7000 50  0001 C CNN "finalized"
@@
 F 0 "C21" H 4265 7046 50  0000 L CNN
 F 1 "0.1uF" H 4265 6955 50  0000 L CNN
-F 2 "Capacitor_SMD:C_0603_1608Metric_Pad1.05x0.95mm_HandSolder" H 4188 6850 50  0001 C CNN
+F 2 "Sonosus:Capacitor_NonPolarizedSmall" H 4188 6850 50  0001 C CNN
 F 3 "~" H 4150 7000 50  0001 C CNN
 F 4 "yes" H 4150 7000 50  0001 C CNN "finalized"
@@
 F 0 "R24" H 4868 5946 50  0000 L CNN
 F 1 "4.7k" H 4868 5855 50  0000 L CNN
-F 2 "Resistor_SMD:R_0603_1608Metric_Pad1.05x0.95mm_HandSolder" V 4840 5890 50  0001 C CNN
+F 2 "Sonosus:Resistor" V 4840 5890 50  0001 C CNN
 F 3 "~" H 4800 5900 50  0001 C CNN
 F 4 "yes" H 4800 5900 50  0001 C CNN "finalized"
@@
 F 0 "R25" H 5268 5946 50  0000 L CNN
 F 1 "4.7k" H 5268 5855 50  0000 L CNN
-F 2 "Resistor_SMD:R_0603_1608Metric_Pad1.05x0.95mm_HandSolder" V 5240 5890 50  0001 C CNN
+F 2 "Sonosus:Resistor" V 5240 5890 50  0001 C CNN
 F 3 "~" H 5200 5900 50  0001 C CNN
 F 4 "yes" H 5200 5900 50  0001 C CNN "finalized"
@@
 F 0 "C22" H 7865 5946 50  0000 L CNN
 F 1 "0.1uF" H 7865 5855 50  0000 L CNN
-F 2 "Capacitor_SMD:C_0603_1608Metric_Pad1.05x0.95mm_HandSolder" H 7788 5750 50  0001 C CNN
+F 2 "Sonosus:Capacitor_NonPolarizedSmall" H 7788 5750 50  0001 C CNN
 F 3 "~" H 7750 5900 50  0001 C CNN
 F 4 "yes" H 7750 5900 50  0001 C CNN "finalized"
@@
 F 0 "C23" H 8415 5946 50  0000 L CNN
 F 1 "10uF" H 8415 5855 50  0000 L CNN
-F 2 "Capacitor_SMD:C_0805_2012Metric_Pad1.15x1.40mm_HandSolder" H 8338 5750 50  0001 C CNN
+F 2 "Capacitor_THT:C_Disc_D4.3mm_W1.9mm_P5.00mm" H 8338 5750 50  0001 C CNN
 F 3 "~" H 8300 5900 50  0001 C CNN
 F 4 "yes & alt" H 8300 5900 50  0001 C CNN "finalized"
@@
 F 0 "C50" H 2815 7046 50  0000 L CNN
 F 1 "0.1uF" H 2815 6955 50  0000 L CNN
-F 2 "Capacitor_SMD:C_0603_1608Metric_Pad1.05x0.95mm_HandSolder" H 2738 6850 50  0001 C CNN
+F 2 "Sonosus:Capacitor_NonPolarizedSmall" H 2738 6850 50  0001 C CNN
 F 3 "~" H 2700 7000 50  0001 C CNN
 F 4 "yes" H 2700 7000 50  0001 C CNN "finalized"
@@
 F 0 "C49" H 2365 7046 50  0000 L CNN
 F 1 "0.1uF" H 2365 6955 50  0000 L CNN
-F 2 "Capacitor_SMD:C_0603_1608Metric_Pad1.05x0.95mm_HandSolder" H 2288 6850 50  0001 C CNN
+F 2 "Sonosus:Capacitor_NonPolarizedSmall" H 2288 6850 50  0001 C CNN
 F 3 "~" H 2250 7000 50  0001 C CNN
 F 4 "yes" H 2250 7000 50  0001 C CNN "finalized"
