File: hardware/mainboard/outputmixer.sch (KiCad schematic (older format))
At the start: 13 parts, among them U14 TL072

Commit message: start to change to tht!
Parts:
- C41, C44: footprint Capacitor_SMD:C_0603_1608Metric_Pad1.05x0.95mm_HandSolder -> Sonosus:Capacitor_NonPolarized
- C45, C46: footprint Capacitor_SMD:C_0603_1608Metric_Pad1.05x0.95mm_HandSolder -> Sonosus:Capacitor_NonPolarizedSmall
- R62, R63, R64, R65, R66, R67, R68, R69: footprint Resistor_SMD:R_0603_1608Metric_Pad1.05x0.95mm_HandSolder -> Sonosus:Resistor
Changed lines of the file:
@@
 F 0 "R64" V 2595 2300 50  0000 C CNN
 F 1 "100k" V 2686 2300 50  0000 C CNN
-F 2 "Resistor_SMD:R_0603_1608Metric_Pad1.05x0.95mm_HandSolder" V 2840 2290 50  0001 C CNN
+F 2 "Sonosus:Resistor" V 2840 2290 50  0001 C CNN
 F 3 "~" H 2800 2300 50  0001 C CNN
 F 4 "1%, 2mW, audio path" H 2800 2300 50  0001 C CNN "Reqs"
@@
 F 0 "R65" V 2900 2500 50  0000 C CNN
 F 1 "100k" V 3000 2500 50  0000 C CNN
-F 2 "Resistor_SMD:R_0603_1608Metric_Pad1.05x0.95mm_HandSolder" V 2840 2490 50  0001 C CNN
+F 2 "Sonosus:Resistor" V 2840 2490 50  0001 C CNN
 F 3 "~" H 2800 2500 50  0001 C CNN
 F 4 "1%, 2mW, audio path" H 2800 2500 50  0001 C CNN "Reqs"
@@
 F 0 "R66" H 3032 2754 50  0000 R CNN
 F 1 "100k" H 3032 2845 50  0000 R CNN
-F 2 "Resistor_SMD:R_0603_1608Metric_Pad1.05x0.95mm_HandSolder" V 3140 2790 50  0001 C CNN
+F 2 "Sonosus:Resistor" V 3140 2790 50  0001 C CNN
 F 3 "~" H 3100 2800 50  0001 C CNN
 F 4 "1%, 2mW, audio path" H 3100 2800 50  0001 C CNN "Reqs"
@@
 F 0 "R67" V 3555 2050 50  0000 C CNN
 F 1 "100k" V 3464 2050 50  0000 C CNN
-F 2 "Resistor_SMD:R_0603_1608Metric_Pad1.05x0.95mm_HandSolder" V 3390 2040 50  0001 C CNN
+F 2 "Sonosus:Resistor" V 3390 2040 50  0001 C CNN
 F 3 "~" H 3350 2050 50  0001 C CNN
 F 4 "1%, 2mW, audio path" H 3350 2050 50  0001 C CNN "Reqs"
@@
 F 0 "R62" V 2750 3700 50  0000 L CNN
 F 1 "100k" V 2550 3650 50  0000 L CNN
-F 2 "Resistor_SMD:R_0603_1608Metric_Pad1.05x0.95mm_HandSolder" V 2690 3740 50  0001 C CNN
+F 2 "Sonosus:Resistor" V 2690 3740 50  0001 C CNN
 F 3 "~" H 2650 3750 50  0001 C CNN
 F 4 "1%, 2mW, audio path" H 2650 3750 50  0001 C CNN "Reqs"
@@
 F 0 "C41" V 3121 1700 50  0000 C CNN
 F 1 "18pF" V 3212 1700 50  0000 C CNN
-F 2 "Capacitor_SMD:C_0603_1608Metric_Pad1.05x0.95mm_HandSolder" H 3350 1700 50  0001 C CNN
+F 2 "Sonosus:Capacitor_NonPolarized" H 3350 1700 50  0001 C CNN
 F 3 "~" H 3350 1700 50  0001 C CNN
 F 4 "yes" H 3350 1700 50  0001 C CNN "finalized"
@@
 F 0 "R63" V 2750 4000 50  0000 L CNN
 F 1 "100k" V 2550 3950 50  0000 L CNN
-F 2 "Resistor_SMD:R_0603_1608Metric_Pad1.05x0.95mm_HandSolder" V 2690 4040 50  0001 C CNN
+F 2 "Sonosus:Resistor" V 2690 4040 50  0001 C CNN
 F 3 "~" H 2650 4050 50  0001 C CNN
 F 4 "1%, 2mW, audio path" H 2650 4050 50  0001 C CNN "Reqs"
@@
 F 0 "R68" V 3605 3800 50  0000 C CNN
 F 1 "100k" V 3514 3800 50  0000 C CNN
-F 2 "Resistor_SMD:R_0603_1608Metric_Pad1.05x0.95mm_HandSolder" V 3440 3790 50  0001 C CNN
+F 2 "Sonosus:Resistor" V 3440 3790 50  0001 C CNN
 F 3 "~" H 3400 3800 50  0001 C CNN
 F 4 "1%, 2mW, audio path" H 3400 3800 50  0001 C CNN "Reqs"
@@
 F 0 "R69" V 4205 4150 50  0000 C CNN
 F 1 "1k" V 4114 4150 50  0000 C CNN
-F 2 "Resistor_SMD:R_0603_1608Metric_Pad1.05x0.95mm_HandSolder" V 4040 4140 50  0001 C CNN
+F 2 "Sonosus:Resistor" V 4040 4140 50  0001 C CNN
 F 3 "~" H 4000 4150 50  0001 C CNN
 F 4 "5%, audio path" H 4000 4150 50  0001 C CNN "Reqs"
@@
 F 0 "C44" V 3171 3450 50  0000 C CNN
 F 1 "18pF" V 3262 3450 50  0000 C CNN
-F 2 "Capacitor_SMD:C_0603_1608Metric_Pad1.05x0.95mm_HandSolder" H 3400 3450 50  0001 C CNN
+F 2 "Sonosus:Capacitor_NonPolarized" H 3400 3450 50  0001 C CNN
 F 3 "~" H 3400 3450 50  0001 C CNN
 F 4 "yes" H 3400 3450 50  0001 C CNN "finalized"
@@
 F 0 "C45" H 6508 3054 50  0000 R CNN
 F 1 "0.1uF" H 6508 3145 50  0000 R CNN
-F 2 "Capacitor_SMD:C_0603_1608Metric_Pad1.05x0.95mm_HandSolder" H 6600 3100 50  0001 C CNN
+F 2 "Sonosus:Capacitor_NonPolarizedSmall" H 6600 3100 50  0001 C CNN
 F 3 "~" H 6600 3100 50  0001 C CNN
 F 4 "yes" H 6600 3100 50  0001 C CNN "finalized"
@@
 F 0 "C46" H 7008 3054 50  0000 R CNN
 F 1 "0.1uF" H 7008 3145 50  0000 R CNN
-F 2 "Capacitor_SMD:C_0603_1608Metric_Pad1.05x0.95mm_HandSolder" H 7100 3100 50  0001 C CNN
+F 2 "Sonosus:Capacitor_NonPolarizedSmall" H 7100 3100 50  0001 C CNN
 F 3 "~" H 7100 3100 50  0001 C CNN
 F 4 "yes" H 7100 3100 50  0001 C CNN "finalized"
